File: r1/src/tr23-sao-r1.kicad_pcb (KiCad board)
At the start: 2 copper layers, 33.5 x 68 mm, 9 parts, among them J1 Conn_02x03_Odd_Even, J2 Wii_Nunchuck_Connector

Commit message: Add fiducials
Parts:
- added FID1: Fiducial, Fiducial:Fiducial_1mm_Mask2mm, B.Cu at (150.0, 116.0)
- added FID2: Fiducial, Fiducial:Fiducial_1mm_Mask2mm, B.Cu at (164.3, 52.5)
Changed lines of the file:
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@@
     )
+  )
+  (footprint "Fiducial:Fiducial_1mm_Mask2mm" (layer "B.Cu")
+    (at 164.3 52.5)
+    (descr "Circular Fiducial, 1mm bare copper, 2mm soldermask opening (Level A)")
+    (tags "fiducial")
+    (property "Sheetfile" "tr23-sao-r1.kicad_sch")
+    (property "Sheetname" "")
+    (property "ki_description" "Fiducial Marker")
+    (property "ki_keywords" "fiducial marker")
+    (attr smd)
+    (fp_text reference "FID2" (at 0 2 180) (layer "B.SilkS") hide
+      (effects (font (size 1 1) (thickness 0.15)) (justify mirror))
+    )
+    (fp_text value "Fiducial" (at 0 -2 180) (layer "B.Fab") hide
+      (effects (font (size 1 1) (thickness 0.15)) (justify mirror))
+    )
+    (fp_circle (center 0 0) (end 1.25 0)
+      (stroke (width 0.05) (type solid)) (fill none) (layer "B.CrtYd"))
+    (fp_circle (center 0 0) (end 1 0)
+      (stroke (width 0.1) (type solid)) (fill none) (layer "B.Fab"))
+    (fp_text user "${REFERENCE}" (at 0 0 180) (layer "B.Fab")
+      (effects (font (size 0.4 0.4) (thickness 0.06)) (justify mirror))
+    )
+    (pad "" smd circle (at 0 0) (size 1 1) (layers "B.Cu" "B.Mask")
+      (solder_mask_margin 0.5) (clearance 0.5))
+  )
+  (footprint "Fiducial:Fiducial_1mm_Mask2mm" (layer "B.Cu")
+    (at 150 116)
+    (descr "Circular Fiducial, 1mm bare copper, 2mm soldermask opening (Level A)")
+    (tags "fiducial")
+    (property "Sheetfile" "tr23-sao-r1.kicad_sch")
+    (property "Sheetname" "")
+    (property "ki_description" "Fiducial Marker")
+    (property "ki_keywords" "fiducial marker")
+    (attr smd)
+    (fp_text reference "FID1" (at 0 2 180) (layer "B.SilkS") hide
+      (effects (font (size 1 1) (thickness 0.15)) (justify mirror))
+    )
+    (fp_text value "Fiducial" (at 0 -2 180) (layer "B.Fab") hide
+      (effects (font (size 1 1) (thickness 0.15)) (justify mirror))
+    )
+    (fp_circle (center 0 0) (end 1.25 0)
+      (stroke (width 0.05) (type solid)) (fill none) (layer "B.CrtYd"))
+    (fp_circle (center 0 0) (end 1 0)
+      (stroke (width 0.1) (type solid)) (fill none) (layer "B.Fab"))
+    (fp_text user "${REFERENCE}" (at 0 0 180) (layer "B.Fab")
+      (effects (font (size 0.4 0.4) (thickness 0.06)) (justify mirror))
+    )
+    (pad "" smd circle (at 0 0) (size 1 1) (layers "B.Cu" "B.Mask")
+      (solder_mask_margin 0.5) (clearance 0.5))
   )
   (footprint "jeffmakes-footprints:LED_RGB_PLCC4_reverse_mount" locked (layer "B.Cu")
@@
     (property "Sheetfile" "tr23-sao-r1.kicad_sch")
     (property "Sheetname" "")
-    (property "dnp" "")
     (property "exclude_from_bom" "")
     (property "ki_description" "RGB LED, red/anode/blue/green")
     (property "ki_keywords" "LED RGB diode")
-    (attr smd exclude_from_pos_files exclude_from_bom dnp)
+    (attr smd exclude_from_pos_files exclude_from_bom)
     (fp_text reference "D1" (at 0 2.4 180) (layer "B.SilkS") hide
       (effects (font (size 1 1) (thickness 0.15)) (justify mirror))

Commit message: Add value to U1
Parts:
- U1: value ~ -> KTD2052A
Changed lines of the file:
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@@
       (effects (font (size 1 1) (thickness 0.15)) (justify mirror))
     )
-    (fp_text value "~" (at 0 -1.95 180) (layer "B.Fab") hide
+    (fp_text value " KTD2052A" (at 0 -1.95 180) (layer "B.Fab") hide
       (effects (font (size 1 1) (thickness 0.15)) (justify mirror))
     )

Commit message: Update value of U1. Update placement data
Parts:
- U1: value KTD2052A -> KTD2052A
Changed lines of the file:
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@@
     (aux_axis_origin 150 105)
     (pcbplotparams
-      (layerselection 0x00010f4_ffffffff)
-      (plot_on_all_layers_selection 0x0000000_00000000)
+      (layerselection 0x0010000_7ffffffe)
+      (plot_on_all_layers_selection 0x0001000_00000000)
       (disableapertmacros false)
       (usegerberextensions false)
@@
       (sketchpadsonfab false)
       (subtractmaskfromsilk true)
-      (outputformat 1)
-      (mirror false)
+      (outputformat 4)
+      (mirror true)
       (drillshape 0)
       (scaleselection 1)
@@
       (effects (font (size 1 1) (thickness 0.15)) (justify mirror))
     )
-    (fp_text value " KTD2052A" (at 0 -1.95 180) (layer "B.Fab") hide
+    (fp_text value "KTD2052A" (at 0 -1.95 180) (layer "B.Fab") hide
       (effects (font (size 1 1) (thickness 0.15)) (justify mirror))
     )

Commit message: Increase board edge-copper clearance to 0.25. Remove drawing sheet title frame from gerbers
Other:
- board text added: "tr23-sao-r1"
Changed lines of the file:
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@@
   (gr_circle (center 146.112132 50.95) (end 146.324264 50.95)
     (stroke (width 0.15) (type default)) (fill none) (layer "B.SilkS"))
+  (gr_text "tr23-sao-r1" (at 142.4 52.15) (layer "B.SilkS")
+    (effects (font (size 0.8 0.8) (thickness 0.15)) (justify left bottom mirror))
+  )
   (gr_text "D1 D3\nD2 D4" (at 164.8 62.4) (layer "B.SilkS")
     (effects (font (size 1 1) (thickness 0.15)) (justify left bottom mirror))
